File: 0003_RGB_Module_WS2812.kicad_sch (KiCad schematic)
At the start: 30 parts

Commit message: Add files via upload
Parts:
- added D16: LED, LED_SMD:LED_0603_1608Metric, symbol Device:LED
- added R1: 470r, Resistor_SMD:R_0603_1608Metric, symbol Device:R
- added U1: ~, Moduler_:pin_header_5-3, symbol moduler_pin:air
- C1, C10, C11, C12, C13, C14, C15, C2, C3, C4, C5, C6, C7, C8, C9: footprint (none) -> Capacitor_SMD:C_0603_1608Metric
Connections:
- net +5V: now also R1.1, U1.7
- net DIN: now also U1.12
- net DOUT: now also U1.13
- net GND: now also D16.1 (K), U1.9
- net at D1.2 (DOUT): now also D2.4 (DIN); no longer D6.4 (DIN)
- net at D3.2 (DOUT): now also D4.4 (DIN); no longer D8.4 (DIN)
- net at D3.4 (DIN): now also D2.2 (DOUT); no longer D12.2 (DOUT)
- net at D12.4 (DIN): now also D11.2 (DOUT); no longer D7.2 (DOUT)
- net at D11.4 (DIN): now also D10.2 (DOUT); no longer D6.2 (DOUT)
- net at D7.4 (DIN): now also D6.2 (DOUT); no longer D2.2 (DOUT)
- net at D15.4 (DIN): now also D14.2 (DOUT); no longer D10.2 (DOUT)
- net at D9.4 (DIN): now also D8.2 (DOUT); no longer D4.2 (DOUT)
- net at D13.2 (DOUT): now also D14.4 (DIN); no longer D4.4 (DIN)
- net at D13.4 (DIN): now also D12.2 (DOUT); no longer D8.2 (DOUT)
- net at D10.4 (DIN): now also D9.2 (DOUT); no longer D5.2 (DOUT)
- net at D5.4 (DIN): now also D4.2 (DOUT); no longer D14.2 (DOUT)
- new net: D16.2 (A), R1.2
- new net: D7.2 (DOUT), D8.4 (DIN)
- new net: D5.2 (DOUT), D6.4 (DIN)
- no-connect marks 0 -> 14
Other:
- note added: "AIR PIN"
- note added: "SENSOR"
- moved on the sheet: C15, C8, D1, D15, D8
